File: _autosave-esp32_io_board.kicad_pcb (KiCad board)
At the start: 2 copper layers, 59 parts, among them J1 USB_B_Micro, J10 Conn_02x04_Counter_Clockwise, J11 Conn_01x02, J12 Conn_01x02, J13 Conn_01x02, J14 Conn_01x02, J15 Conn_01x02, J16 Conn_01x02, J17 Conn_01x02, J18 Conn_01x02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

Commit message: initial layout without traces
Parts:
- D2: footprint Diode_SMD:D_SOD-323F -> Diode_SMD:D_SOD-123F
- D7: footprint LED_SMD:LED_RGB_5050-6 -> LED_SMD:LED_0603_1608Metric
- moved R6 88.6 mm to (173.2, 87.6), turned to 180 degrees
- moved C8 88.2 mm to (173.2, 85.9)
- moved C3 86.1 mm to (169.2, 95.5), turned to 180 degrees
- moved J3 79.3 mm to (173.0, 90.9), turned to 90 degrees
- moved C5 79.2 mm to (169.2, 103.1)
- moved C6 78.6 mm to (175.5, 103.1)
- moved C4 77.8 mm to (175.5, 95.5), turned to 180 degrees
- moved SW1 71.8 mm to (166.1, 88.9), turned to 270 degrees
- moved J11 70.7 mm to (180.6, 126.7), turned to 180 degrees
- moved J18 69.0 mm to (188.5, 116.1)
- moved U2 67.8 mm to (172.0, 99.3)
- moved D3 67.4 mm to (177.8, 113.0), turned to 180 degrees
- moved D6 66.1 mm to (168.9, 113.0), turned to 180 degrees
- moved R10 65.7 mm to (194.8, 122.2)
- moved J5 65.3 mm to (178.3, 119.1), turned to 270 degrees
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