File: esp32_io_board.sch (KiCad schematic (older format))
At the start: 66 parts, among them J1 USB_B_Micro, J11 Conn_01x02, J12 Conn_01x02, J13 Conn_01x02, J14 Conn_01x02, J2 Conn_02x04_Counter_Clockwise, J3 Conn_01x02, J4 Conn_01x04, J5 RASPBERRYPI-40-PIN-GPIO, J7 Conn_01x02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

Commit message: layout
Parts:
- removed D3, D6: LED_RGB, LED_SMD:LED_RGB_5050-6, symbol Device:LED_RGB
- removed J4: Conn_01x04, Connector_PinHeader_2.54mm:PinHeader_1x04_P2.54mm_Vertical, symbol Connector_Generic:Conn_01x04
- added J4: Conn_01x02, Connector_PinHeader_2.54mm:PinHeader_1x02_P2.54mm_Vertical, symbol Connector_Generic:Conn_01x02
- added R13, R14, R15, R16: R_Small, Resistor_SMD:R_0603_1608Metric, symbol Device:R_Small
- R12: renamed from R?; footprint (none) -> Resistor_SMD:R_0603_1608Metric
- U7: renamed from U?; footprint (none) -> Package_SO:SOIC-8-1EP_3.9x4.9mm_P1.27mm_EP2.35x2.35mm
- gave numbers to parts that had none: 6
Connections:
- net 3.3V is gone; now on net +3V3: C6.1
- net +3V3: now also R13.2, R14.2, R15.1, R16.1
- net at U4.23 (IO15), U6.23 (SDA): now also R13.1
- net at U4.24 (IO2), U6.22 (SCL): now also R14.1
- net at JP8.2 (B), U6.18 (SC6): now also R15.2
- net at JP9.2 (B), U6.17 (SD6): now also R16.2
- net ci: no longer names the net of U4.16 (IO13)
- net ci: now also J4.1 (Pin_1)
- net di: no longer names the net of U4.14 (IO12)
- net di: now also J4.2 (Pin_2)

Commit message: layout update
Parts:
- removed C3, C4, C5, C6: C_Small, Capacitor_SMD:C_0603_1608Metric, symbol Device:C_Small
- removed JP5, JP6: SolderJumper_2_Open, Jumper:SolderJumper-2_P1.3mm_Open_RoundedPad1.0x1.5mm, symbol Jumper:SolderJumper_2_Open
- removed U2, U3: TXB0104PW, Package_SO:TSSOP-14_4.4x5mm_P0.65mm, symbol Logic_LevelTranslator:TXB0104PW
Connections:
- net pin10 is gone; now on an unnamed net: U4.10 (IO25)
- net pin11 is gone; now on an unnamed net: U4.11 (IO26)
- net pin12 is gone; now on an unnamed net: U4.12 (IO27)
- net pin13 is gone; now on an unnamed net: U4.13 (IO14)
- net pin6 is gone; now on an unnamed net: U4.6 (IO34)
- net pin7 is gone; now on an unnamed net: U4.7 (IO35)
- net pin8 is gone; now on an unnamed net: U4.8 (IO32)
- net pin9 is gone; now on an unnamed net: U4.9 (IO33)
- net +5V: no longer J7.1 (Pin_1)
- net GND: now also U7.1 (A0), U7.2 (A1), U7.3 (A2), U7.4 (GND)
- net VCC: now also J7.1 (Pin_1)
- no-connect marks 34 -> 40
Other:
- moved on the sheet: J2
