File: portia.sch (KiCad schematic (older format))
At the start: 16 parts, among them J1 Conn_01x02, J2 Conn_01x02, J3 Conn_02x08_Odd_Even, J5 Conn_02x08_Odd_Even, SW1 Reset, SW2 Reset, U4 ESP32-WROOM

Commit message: update layout
Parts:
- removed J3, J5: Conn_02x08_Odd_Even, Connector_PinHeader_2.54mm:PinHeader_2x08_P2.54mm_Vertical, symbol Connector_Generic:Conn_02x08_Odd_Even
- added J? (x2): Conn_02x11_Odd_Even, symbol Connector_Generic:Conn_02x11_Odd_Even
Connections:
- wire segments 182 -> 211
Changed lines of the file:
@@
 L power:+3.3V #PWR0102
 U 1 1 5BF2CD9B
-P 8100 4750
-F 0 "#PWR0102" H 8100 4600 50  0001 C CNN
-F 1 "+3.3V" H 8115 4923 50  0000 C CNN
-F 2 "" H 8100 4750 50  0001 C CNN
-F 3 "" H 8100 4750 50  0001 C CNN
-	1    8100 4750
+P 8100 4350
+F 0 "#PWR0102" H 8100 4200 50  0001 C CNN
+F 1 "+3.3V" H 8115 4523 50  0000 C CNN
+F 2 "" H 8100 4350 50  0001 C CNN
+F 3 "" H 8100 4350 50  0001 C CNN
+	1    8100 4350
 	1    0    0    -1
 $EndComp
@@
 $EndComp
 Wire Wire Line
-	8100 4750 8100 5300
-Wire Wire Line
 	8100 5300 9150 5300
 Wire Wire Line
-	9150 5500 7600 5500
-Wire Wire Line
-	7550 5600 7650 5600
-Wire Wire Line
 	7550 5800 7850 5800
 Wire Wire Line
@@
 Wire Wire Line
 	7550 6200 7650 6200
-Wire Wire Line
-	11000 5550 11200 5550
 Wire Wire Line
 	11000 6450 11000 6550
@@
 	11000 6250 11450 6250
 Wire Wire Line
-	11000 5150 11400 5150
-Wire Wire Line
-	11000 5350 11300 5350
-Wire Wire Line
-	11500 5450 11250 5450
-Wire Wire Line
-	11500 5650 11300 5650
+	12000 5650 11300 5650
 Wire Wire Line
 	11150 5650 11150 5750
@@
 	11150 5750 11000 5750
 Wire Wire Line
-	11500 5750 11350 5750
+	12000 5750 11350 5750
 Wire Wire Line
 	11200 5850 11000 5850
 Wire Wire Line
-	11500 5850 11400 5850
+	12000 5850 11400 5850
 Wire Wire Line
 	11250 5850 11250 5950
@@
 	11250 5950 11000 5950
 Wire Wire Line
-	11400 5150 11400 4900
-Wire Wire Line
-	11400 4900 12000 4900
-Wire Wire Line
-	12000 4900 12000 5150
-Connection ~ 11400 5150
-Wire Wire Line
-	11400 5150 11500 5150
-Wire Wire Line
-	12050 4850 12050 5250
-Wire Wire Line
-	12050 5250 12000 5250
-Wire Wire Line
-	11350 4850 11350 5250
-Wire Wire Line
-	11350 4850 12050 4850
-Connection ~ 11350 5250
-Wire Wire Line
-	11350 5250 11500 5250
-Wire Wire Line
-	11000 5250 11350 5250
-Wire Wire Line
-	11300 5350 11300 4800
-Wire Wire Line
-	11300 4800 12100 4800
-Connection ~ 11300 5350
-Wire Wire Line
-	11300 5350 11500 5350
-Wire Wire Line
-	12100 4800 12100 5350
-Wire Wire Line
-	12100 5350 12000 5350
-Wire Wire Line
-	11250 5450 11250 4750
-Wire Wire Line
-	11250 4750 12150 4750
-Wire Wire Line
-	12150 4750 12150 5450
-Wire Wire Line
-	12150 5450 12000 5450
-Connection ~ 11250 5450
-Wire Wire Line
-	11250 5450 11000 5450
-Wire Wire Line
-	11200 5550 11200 4700
-Wire Wire Line
-	11200 4700 12200 4700
-Connection ~ 11200 5550
-Wire Wire Line
-	11200 5550 11500 5550
-Wire Wire Line
-	12200 4700 12200 5550
-Wire Wire Line
-	12200 5550 12000 5550
+	12550 5250 12500 5250
+Wire Wire Line
+	12600 5350 12500 5350
+Wire Wire Line
+	12650 5450 12500 5450
+Wire Wire Line
+	12700 5550 12500 5550
 Wire Wire Line
 	11200 5750 11200 5850
 Wire Wire Line
 	11400 5850 11400 6000
-Wire Wire Line
-	11400 6000 12000 6000
-Wire Wire Line
-	12000 6000 12000 5850
 Connection ~ 11400 5850
 Wire Wire Line
@@
 Wire Wire Line
 	11350 5750 11350 6050
-Wire Wire Line
-	11350 6050 12050 6050
 Connection ~ 11350 5750
 Wire Wire Line
 	11350 5750 11200 5750
 Wire Wire Line
-	12050 6050 12050 5750
-Wire Wire Line
-	12050 5750 12000 5750
-Wire Wire Line
 	11300 5650 11300 6100
-Wire Wire Line
-	11300 6100 12100 6100
 Connection ~ 11300 5650
 Wire Wire Line
 	11300 5650 11150 5650
-Wire Wire Line
-	12100 6100 12100 5650
-Wire Wire Line
-	12100 5650 12000 5650
 Wire Wire Line
 	9150 5700 7900 5700
@@
 Wire Wire Line
 	6800 5700 6800 6600
-Wire Wire Line
-	7050 5500 7050 5300
-Wire Wire Line
-	7050 5300 7600 5300
-Wire Wire Line
-	7600 5300 7600 5500
-Connection ~ 7600 5500
-Wire Wire Line
-	7600 5500 7550 5500
-Wire Wire Line
-	7000 5250 7000 5600
-Wire Wire Line
-	7000 5600 7050 5600
-Wire Wire Line
-	7650 5250 7650 5600
-Connection ~ 7650 5600
-Wire Wire Line
-	7650 5600 9150 5600
 Wire Wire Line
 	9150 6300 8400 6300
@@
 Wire Wire Line
 	8600 7250 8600 7500
-Wire Wire Line
-	7000 5250 7650 5250
-$Comp
-L power:GND #PWR0106
-U 1 1 5CB85C38
-P 6050 4750
-F 0 "#PWR0106" H 6050 4500 50  0001 C CNN
-F 1 "GND" V 6055 4622 50  0000 R CNN
-F 2 "" H 6050 4750 50  0001 C CNN
-F 3 "" H 6050 4750 50  0001 C CNN
-	1    6050 4750
-	1    0    0    -1
-$EndComp
 Wire Wire Line
 	6150 4500 6150 4900
@@
 	11000 7700 11150 7700
 $Comp
-L Connector_Generic:Conn_02x08_Odd_Even J3
-U 1 1 5C751B37
-P 7250 5800
-F 0 "J3" H 7300 6317 50  0000 C CNN
-F 1 "Conn_02x08_Odd_Even" H 7300 6226 50  0000 C CNN
-F 2 "Connector_PinHeader_2.54mm:PinHeader_2x08_P2.54mm_Vertical" H 7250 5800 50  0001 C CNN
-F 3 "~" H 7250 5800 50  0001 C CNN
-	1    7250 5800
-	1    0    0    -1
-$EndComp
-$Comp
-L Connector_Generic:Conn_02x08_Odd_Even J5
-U 1 1 5C75C447
-P 11800 5550
-F 0 "J5" H 11850 4925 50  0000 C CNN
-F 1 "Conn_02x08_Odd_Even" H 11850 5016 50  0000 C CNN
-F 2 "Connector_PinHeader_2.54mm:PinHeader_2x08_P2.54mm_Vertical" H 11800 5550 50  0001 C CNN
-F 3 "~" H 11800 5550 50  0001 C CNN
-	1    11800 5550
-	-1   0    0    1
-$EndComp
-$Comp
 L Connector_Generic:Conn_02x06_Odd_Even J?
 U 1 1 5C7B3D0C
@@
 	0    -1   -1   0
 $EndComp
+$Comp
+L Connector_Generic:Conn_02x11_Odd_Even J?
+U 1 1 5C751064
+P 7250 5700
+F 0 "J?" H 7300 6417 50  0000 C CNN
+F 1 "Conn_02x11_Odd_Even" H 7300 6326 50  0000 C CNN
+F 2 "" H 7250 5700 50  0001 C CNN
+F 3 "~" H 7250 5700 50  0001 C CNN
+	1    7250 5700
+	1    0    0    -1
+$EndComp
+Wire Wire Line
+	7550 5600 7900 5600
+Wire Wire Line
+	7050 5600 6800 5600
+Wire Wire Line
+	6800 5600 6800 4900
+Wire Wire Line
+	6800 4900 7900 4900
+Wire Wire Line
+	7550 5500 7850 5500
+Wire Wire Line
+	7900 4900 7900 5600
+Connection ~ 7900 5600
+Wire Wire Line
+	7900 5600 9150 5600
+Wire Wire Line
+	6850 5500 7050 5500
+Wire Wire Line
+	6850 5500 6850 4950
+Wire Wire Line
+	7850 4950 7850 5500
+Wire Wire Line
+	6850 4950 7850 4950
+Connection ~ 7850 5500
+Wire Wire Line
+	7850 5500 9150 5500
+$Comp
+L power:GND #PWR0106
+U 1 1 5CB85C38
+P 7550 4350
+F 0 "#PWR0106" H 7550 4100 50  0001 C CNN
+F 1 "GND" V 7555 4222 50  0000 R CNN
+F 2 "" H 7550 4350 50  0001 C CNN
+F 3 "" H 7550 4350 50  0001 C CNN
+	1    7550 4350
+	-1   0    0    1
+$EndComp
+Wire Wire Line
+	7550 4350 7550 4600
+Wire Wire Line
+	7050 5200 7050 4600
+Wire Wire Line
+	7050 4600 7550 4600
+Connection ~ 7550 4600
+Wire Wire Line
+	7550 4600 7550 5200
+Wire Wire Line
+	8100 5300 7650 5300
+Connection ~ 8100 5300
+Wire Wire Line
+	7650 5300 7650 5400
+Wire Wire Line
+	7650 5400 7550 5400
+Connection ~ 7650 5300
+Wire Wire Line
+	7650 5300 7550 5300
+Wire Wire Line
+	7050 5300 6500 5300
+Wire Wire Line
+	7050 5400 6500 5400
+Wire Wire Line
+	6500 5400 6500 5300
+Wire Wire Line
+	6500 4850 8100 4850
+Connection ~ 6500 5300
+Wire Wire Line
+	6500 5300 6500 4850
+Connection ~ 8100 4850
+Wire Wire Line
+	8100 4850 8100 5300
+Wire Wire Line
+	8100 4350 8100 4850
+Wire Wire Line
+	12700 3450 12700 5550
+Wire Wire Line
+	11200 3450 12700 3450
+Wire Wire Line
+	11200 5550 12000 5550
+Wire Wire Line
+	11000 5550 11200 5550
+Connection ~ 11200 5550
+Wire Wire Line
+	11200 5550 11200 3450
+Wire Wire Line
+	12650 3500 12650 5450
+Wire Wire Line
+	11250 3500 12650 3500
+Wire Wire Line
+	11250 5450 11000 5450
+Wire Wire Line
+	12000 5450 11250 5450
+Connection ~ 11250 5450
+Wire Wire Line
+	11250 5450 11250 3500
+Wire Wire Line
+	12600 3550 12600 5350
+Wire Wire Line
+	11300 3550 12600 3550
+Wire Wire Line
+	11300 5350 12000 5350
+Wire Wire Line
+	11000 5350 11300 5350
+Connection ~ 11300 5350
+Wire Wire Line
+	11300 5350 11300 3550
+Wire Wire Line
+	11350 3600 12550 3600
+Wire Wire Line
+	11000 5250 11350 5250
+Wire Wire Line
+	11350 5250 12000 5250
+Connection ~ 11350 5250
+Wire Wire Line
+	11350 3600 11350 5250
+Wire Wire Line
+	12550 3600 12550 5250
+Wire Wire Line
+	11400 5150 12000 5150
+Wire Wire Line
+	11000 5150 11400 5150
+Connection ~ 11400 5150
+Wire Wire Line
+	11400 5150 11400 3650
+$Comp
+L Connector_Generic:Conn_02x11_Odd_Even J?
+U 1 1 5C9C366B
+P 12200 5350
+F 0 "J?" H 12250 6067 50  0000 C CNN
+F 1 "Conn_02x11_Odd_Even" H 12250 5976 50  0000 C CNN
+F 2 "" H 12200 5350 50  0001 C CNN
+F 3 "~" H 12200 5350 50  0001 C CNN
+	1    12200 5350
+	1    0    0    -1
+$EndComp
+Wire Wire Line
+	12500 5150 13950 5150
+Wire Wire Line
+	13950 5150 13950 3650
+Wire Wire Line
+	11400 3650 13950 3650
+Wire Wire Line
+	12500 4950 13150 4950
+Wire Wire Line
+	13150 4950 13150 4700
+Wire Wire Line
+	13150 4550 11900 4550
+Wire Wire Line
+	11900 4550 11900 4950
+Wire Wire Line
+	11900 4950 12000 4950
+Wire Wire Line
+	12500 5050 13200 5050
+Wire Wire Line
+	13200 4500 13200 4950
+Wire Wire Line
+	11850 4500 13200 4500
+Wire Wire Line
+	11850 4500 11850 5050
+Wire Wire Line
+	11850 5050 12000 5050
+Wire Wire Line
+	12000 4600 12000 4850
+Wire Wire Line
+	12000 4600 12100 4600
+Wire Wire Line
+	12500 4600 12500 4850
+Connection ~ 12100 4600
+Wire Wire Line
+	12100 4600 12500 4600
+Wire Wire Line
+	12100 3100 12100 4600
+Wire Wire Line
+	13150 4700 13500 4700
+Connection ~ 13150 4700
+Wire Wire Line
+	13150 4700 13150 4550
+Wire Wire Line
+	13500 4700 13500 4950
+Wire Wire Line
+	13500 4950 13200 4950
+Connection ~ 13500 4700
+Wire Wire Line
+	13500 4700 14350 4700
+Connection ~ 13200 4950
+Wire Wire Line
+	13200 4950 13200 5050
 $EndSCHEMATC
