File: portia.sch (KiCad schematic (older format))
At the start: 16 parts, among them J1 Conn_01x02, J2 Conn_01x02, SW1 Reset, SW2 Reset, U4 ESP32-WROOM

Commit message: update layout
Parts:
- removed J1, J2: Conn_01x02, Connector_PinHeader_2.54mm:PinHeader_1x02_P2.54mm_Vertical, symbol Connector_Generic:Conn_01x02
- removed J? (x2): Conn_02x11_Odd_Even, symbol Connector_Generic:Conn_02x11_Odd_Even
- removed J?: Conn_02x06_Odd_Even, symbol Connector_Generic:Conn_02x06_Odd_Even
- added J1, J2: Conn_01x11, symbol Connector_Generic:Conn_01x11
Connections:
- wire segments 211 -> 73

Commit message: add castellated footprint
Parts:
- removed D1: LED_ARGB, LED_SMD:LED_RGB_1210, symbol Device:LED_ARGB
- removed R1: R10, Resistor_SMD:R_0603_1608Metric, symbol Device:R
- removed R2, R3: R60, Resistor_SMD:R_0603_1608Metric, symbol Device:R
Connections:
- wire segments 73 -> 66
Changed lines of the file:
@@
 Wire Wire Line
 	11200 6150 11200 7200
-$Comp
-L Device:LED_ARGB D1
-U 1 1 5CCFD356
-P 10650 8950
-F 0 "D1" V 10604 9310 50  0000 L CNN
-F 1 "LED_ARGB" V 10695 9310 50  0000 L CNN
-F 2 "LED_SMD:LED_RGB_1210" H 10650 8900 50  0001 C CNN
-F 3 "~" H 10650 8900 50  0001 C CNN
-	1    10650 8950
-	0    1    1    0
-$EndComp
-Wire Wire Line
-	11450 8750 10850 8750
 Wire Wire Line
 	11700 7300 11700 9250
@@
 Wire Wire Line
 	11700 9250 11700 9800
-$Comp
-L Device:R R3
-U 1 1 5CD71E2E
-P 11450 8250
-F 0 "R3" V 11350 8250 50  0000 C CNN
-F 1 "R60" V 11550 8250 50  0000 C CNN
-F 2 "Resistor_SMD:R_0603_1608Metric" V 11380 8250 50  0001 C CNN
-F 3 "~" H 11450 8250 50  0001 C CNN
-	1    11450 8250
-	-1   0    0    1
-$EndComp
-$Comp
-L Device:R R2
-U 1 1 5CD73029
-P 10650 8250
-F 0 "R2" V 10550 8250 50  0000 C CNN
-F 1 "R60" V 10450 8250 50  0000 C CNN
-F 2 "Resistor_SMD:R_0603_1608Metric" V 10580 8250 50  0001 C CNN
-F 3 "~" H 10650 8250 50  0001 C CNN
-	1    10650 8250
-	-1   0    0    1
-$EndComp
-$Comp
-L Device:R R1
-U 1 1 5CD731D2
-P 10450 8250
-F 0 "R1" V 10350 8250 50  0000 C CNN
-F 1 "R10" V 10550 8250 50  0000 C CNN
-F 2 "Resistor_SMD:R_0603_1608Metric" V 10380 8250 50  0001 C CNN
-F 3 "~" H 10450 8250 50  0001 C CNN
-	1    10450 8250
-	-1   0    0    1
-$EndComp
-Wire Wire Line
-	11450 8400 11450 8750
-Wire Wire Line
-	10650 8100 10650 7050
 Wire Wire Line
 	10650 7050 10550 7050
@@
 	10550 6950 10550 7050
 Wire Wire Line
-	10650 8400 10650 8750
-Wire Wire Line
-	11450 6250 11450 8100
-Wire Wire Line
-	10450 6950 10450 8100
-Wire Wire Line
-	10450 8400 10450 8750
-Wire Wire Line
 	11000 7700 11150 7700

Commit message: update layout
Parts:
- added C1, C2: C_Small, Capacitor_SMD:C_0603_1608Metric_Pad1.05x0.95mm_HandSolder, symbol Device:C_Small
- added J3: Conn_01x02, Connector_PinHeader_2.54mm:PinHeader_1x11_P2.54mm_Vertical, symbol Connector_Generic:Conn_01x02
- added J4: Conn_02x06_Odd_Even, sb_designed_footprints:castellated12, symbol Connector_Generic:Conn_02x06_Odd_Even
- added U1: LM1117-3.3, Package_TO_SOT_SMD:SOT-223, symbol Regulator_Linear:LM1117-3.3
- J1, J2: footprint (none) -> Connector_PinHeader_2.54mm:PinHeader_1x11_P2.54mm_Vertical
Connections:
- net labels added: +5V
- wire segments 66 -> 92

Commit message: update layout
Parts:
- removed C1, C2: C_Small, Capacitor_SMD:C_0603_1608Metric_Pad1.05x0.95mm_HandSolder, symbol Device:C_Small
- removed J1, J2: Conn_01x11, Connector_PinHeader_2.54mm:PinHeader_1x11_P2.54mm_Vertical, symbol Connector_Generic:Conn_01x11
- removed J4: Conn_02x06_Odd_Even, sb_designed_footprints:castellated12, symbol Connector_Generic:Conn_02x06_Odd_Even
- removed U1: LM1117-3.3, Package_TO_SOT_SMD:SOT-223, symbol Regulator_Linear:LM1117-3.3
- added J1: Conn_01x02, Connector_PinHeader_2.54mm:PinHeader_1x02_P2.54mm_Vertical, symbol Connector_Generic:Conn_01x02
- added J2, J5: Conn_01x08, Connector_PinHeader_2.54mm:PinHeader_1x08_P2.54mm_Vertical, symbol Connector_Generic:Conn_01x08
- added J4: Conn_02x08_Counter_Clockwise, sb_designed_footprints:castellated12, symbol Connector_Generic:Conn_02x08_Counter_Clockwise
- H1, H5: footprint MountingHole:MountingHole_3mm -> sb_designed_footprints:MountingHole_3mm
- J3: footprint Connector_PinHeader_2.54mm:PinHeader_1x11_P2.54mm_Vertical -> Connector_PinHeader_2.54mm:PinHeader_1x02_P2.54mm_Vertical
Connections:
- net +5V is gone; now on net +3V3: J3.1 (Pin_1)
- net +3V3: now also J1.1 (Pin_1), J4.10 (Pin_10), J4.2 (Pin_2), J4.4 (Pin_4)
- net GND: now also J1.2 (Pin_2), J4.1 (Pin_1), J4.11 (Pin_11), J4.3 (Pin_3)
- net at U4.10 (IO25): now also J2.2 (Pin_2)
- net at U4.11 (IO26): now also J2.1 (Pin_1)
- net at U4.12 (IO27): now also J4.5 (Pin_5)
- net at U4.13 (IO14): now also J4.6 (Pin_6)
- net at U4.14 (IO12): now also J4.7 (Pin_7)
- net at U4.16 (IO13): now also J4.8 (Pin_8)
- net at U4.23 (IO15): now also J4.16 (Pin_16)
- net at U4.24 (IO2): now also J4.15 (Pin_15)
- net at U4.26 (IO4): now also J4.14 (Pin_14)
- net at U4.27 (IO16): now also J4.13 (Pin_13)
- net at U4.28 (IO17): now also J4.12 (Pin_12)
- net at U4.29 (IO5): now also J5.8 (Pin_8)
- net at U4.30 (IO18): now also J5.7 (Pin_7)
- net at U4.31 (IO19): now also J5.6 (Pin_6)
- net at U4.33 (IO21): now also J5.5 (Pin_5)
- net at U4.34 (RXD0): now also J5.4 (Pin_4)
- net at U4.35 (TXD0): now also J5.3 (Pin_3)
- net at U4.36 (IO22): now also J5.2 (Pin_2)
- net at U4.37 (IO23): now also J5.1 (Pin_1)
- net at U4.4 (SENSOR_VP): now also J2.8 (Pin_8)
- net at U4.5 (SENSOR_VN): now also J2.7 (Pin_7)
- net at U4.6 (IO34): now also J2.6 (Pin_6)
- net at U4.7 (IO35): now also J2.5 (Pin_5)
- net at U4.8 (IO32): now also J2.4 (Pin_4)
- net at U4.9 (IO33): now also J2.3 (Pin_3)
- no-connect marks 7 -> 8
Other:
- moved on the sheet: J3

Commit message: update layout
Parts:
- removed J1, J3: Conn_01x02, Connector_PinHeader_2.54mm:PinHeader_1x02_P2.54mm_Vertical, symbol Connector_Generic:Conn_01x02
- added H2, H3: MountingHole, sb_designed_footprints:MountingHole_3mm, symbol Mechanical:MountingHole
- added J6: Conn_02x06_Counter_Clockwise, Connector_PinHeader_2.54mm:PinHeader_2x06_P2.54mm_Vertical, symbol Connector_Generic:Conn_02x06_Counter_Clockwise
- Boot1: renamed from SW2; value Reset -> Boot_ESP
- Reset1: renamed from SW1; value Reset -> EN
Connections:
- net +3V3: now also J6.2 (Pin_2), J6.8 (Pin_8)
- net GND: now also J6.1 (Pin_1), J6.10 (Pin_10), J6.3 (Pin_3), J6.4 (Pin_4), J6.5 (Pin_5), J6.6 (Pin_6), J6.7 (Pin_7), J6.9 (Pin_9)
- net at J4.13 (Pin_13), U4.27 (IO16): now also J6.12 (Pin_12)
- net at J4.12 (Pin_12), U4.28 (IO17): now also J6.11 (Pin_11)
Changed lines of the file:
@@
 $EndComp
 $Comp
-L Switch:SW_Push SW1
+L Switch:SW_Push Reset1
 U 1 1 5C8C98D8
 P 8900 4450
-F 0 "SW1" H 8900 4735 50  0000 C CNN
-F 1 "Reset" H 8900 4644 50  0000 C CNN
+F 0 "Reset1" H 8900 4735 50  0000 C CNN
+F 1 "EN" H 8900 4644 50  0000 C CNN
 F 2 "Button_Switch_SMD:SW_SPST_B3U-1000P-B" H 8900 4650 50  0001 C CNN
 F 3 "" H 8900 4650 50  0001 C CNN
@@
 P 3450 7500
 F 0 "H5" H 3550 7546 50  0000 L CNN
-F 1 "MountingHole" H 3750 7500 50  0000 L CNN
+F 1 "MountingHole" H 3750 7800 50  0000 L CNN
 F 2 "sb_designed_footprints:MountingHole_3mm" H 3450 7500 50  0001 C CNN
 F 3 "~" H 3450 7500 50  0001 C CNN
@@
 P 3450 7200
 F 0 "H1" H 3550 7246 50  0000 L CNN
-F 1 "MountingHole" H 3750 7200 50  0000 L CNN
+F 1 "MountingHole" H 3750 7300 50  0000 L CNN
 F 2 "sb_designed_footprints:MountingHole_3mm" H 3450 7200 50  0001 C CNN
 F 3 "~" H 3450 7200 50  0001 C CNN
@@
 	11700 6650 11700 7000
 $Comp
-L Switch:SW_Push SW2
+L Switch:SW_Push Boot1
 U 1 1 5C773290
 P 12850 6650
-F 0 "SW2" H 12850 6935 50  0000 C CNN
-F 1 "Reset" H 12850 6844 50  0000 C CNN
+F 0 "Boot1" H 12850 6935 50  0000 C CNN
+F 1 "Boot_ESP" H 12850 6844 50  0000 C CNN
 F 2 "Button_Switch_SMD:SW_SPST_B3U-1000P-B" H 12850 6850 50  0001 C CNN
 F 3 "" H 12850 6850 50  0001 C CNN
@@
 L power:+3.3V #PWR0104
 U 1 1 5C775CD3
-P 11700 9800
-F 0 "#PWR0104" H 11700 9650 50  0001 C CNN
-F 1 "+3.3V" H 11715 9973 50  0000 C CNN
-F 2 "" H 11700 9800 50  0001 C CNN
-F 3 "" H 11700 9800 50  0001 C CNN
-	1    11700 9800
+P 11700 10300
+F 0 "#PWR0104" H 11700 10150 50  0001 C CNN
+F 1 "+3.3V" H 11715 10473 50  0000 C CNN
+F 2 "" H 11700 10300 50  0001 C CNN
+F 3 "" H 11700 10300 50  0001 C CNN
+	1    11700 10300
 	-1   0    0    1
 $EndComp
@@
 	9500 6950 9500 7700
 Wire Wire Line
-	11700 7300 11700 9800
+	11700 7300 11700 9650
 Wire Wire Line
 	11000 7700 12500 7700
@@
 $EndComp
 $Comp
-L Connector_Generic:Conn_01x02 J3
-U 1 1 5C7E3667
-P 7050 3600
-F 0 "J3" V 7016 3412 50  0000 R CNN
-F 1 "Conn_01x02" V 6925 3412 50  0000 R CNN
-F 2 "Connector_PinHeader_2.54mm:PinHeader_1x02_P2.54mm_Vertical" H 7050 3600 50  0001 C CNN
-F 3 "~" H 7050 3600 50  0001 C CNN
-	1    7050 3600
-	0    -1   -1   0
-$EndComp
-Wire Wire Line
-	7050 3800 7050 4250
-Wire Wire Line
-	7150 3800 7150 4450
-$Comp
-L power:GND #PWR0118
-U 1 1 5C80E4FE
-P 7150 4450
-F 0 "#PWR0118" H 7150 4200 50  0001 C CNN
-F 1 "GND" V 7155 4322 50  0000 R CNN
-F 2 "" H 7150 4450 50  0001 C CNN
-F 3 "" H 7150 4450 50  0001 C CNN
-	1    7150 4450
-	-1   0    0    -1
-$EndComp
-$Comp
 L Connector_Generic:Conn_01x08 J2
 U 1 1 5C8239F2
@@
 Connection ~ 11000 6550
 $Comp
-L power:+3.3V #PWR0106
-U 1 1 5C85FFF8
-P 7050 4250
-F 0 "#PWR0106" H 7050 4100 50  0001 C CNN
-F 1 "+3.3V" H 7065 4423 50  0000 C CNN
-F 2 "" H 7050 4250 50  0001 C CNN
-F 3 "" H 7050 4250 50  0001 C CNN
-	1    7050 4250
-	-1   0    0    1
-$EndComp
-$Comp
-L Connector_Generic:Conn_01x02 J1
-U 1 1 5C86377F
-P 6250 3600
-F 0 "J1" V 6216 3412 50  0000 R CNN
-F 1 "Conn_01x02" V 6125 3412 50  0000 R CNN
-F 2 "Connector_PinHeader_2.54mm:PinHeader_1x02_P2.54mm_Vertical" H 6250 3600 50  0001 C CNN
-F 3 "~" H 6250 3600 50  0001 C CNN
-	1    6250 3600
-	0    -1   -1   0
-$EndComp
-Wire Wire Line
-	6250 3800 6250 4250
-Wire Wire Line
-	6350 3800 6350 4450
-$Comp
-L power:GND #PWR0107
-U 1 1 5C863787
-P 6350 4450
-F 0 "#PWR0107" H 6350 4200 50  0001 C CNN
-F 1 "GND" V 6355 4322 50  0000 R CNN
-F 2 "" H 6350 4450 50  0001 C CNN
-F 3 "" H 6350 4450 50  0001 C CNN
-	1    6350 4450
-	-1   0    0    -1
-$EndComp
-$Comp
 L power:+3.3V #PWR0109
 U 1 1 5C86378D
-P 6250 4250
-F 0 "#PWR0109" H 6250 4100 50  0001 C CNN
-F 1 "+3.3V" H 6265 4423 50  0000 C CNN
-F 2 "" H 6250 4250 50  0001 C CNN
-F 3 "" H 6250 4250 50  0001 C CNN
-	1    6250 4250
-	-1   0    0    1
+P 9100 9350
+F 0 "#PWR0109" H 9100 9200 50  0001 C CNN
+F 1 "+3.3V" H 9115 9523 50  0000 C CNN
+F 2 "" H 9100 9350 50  0001 C CNN
+F 3 "" H 9100 9350 50  0001 C CNN
+	1    9100 9350
+	0    -1   -1   0
 $EndComp
 $Comp
@@
 	10450 8400 11300 8400
 Wire Wire Line
-	11200 8500 10450 8500
+	11200 8500 10550 8500
 Wire Wire Line
 	11200 6150 11200 8500
 Wire Wire Line
-	11250 8600 10450 8600
+	11250 8600 10650 8600
 Wire Wire Line
 	11250 6050 11250 8600
@@
 Wire Wire Line
 	9950 8600 8500 8600
+$Comp
+L Mechanical:MountingHole H2
+U 1 1 5C845D8D
+P 3450 7800
+F 0 "H2" H 3550 7846 50  0000 L CNN
+F 1 "MountingHole" H 3750 8300 50  0000 L CNN
+F 2 "sb_designed_footprints:MountingHole_3mm" H 3450 7800 50  0001 C CNN
+F 3 "~" H 3450 7800 50  0001 C CNN
+	1    3450 7800
+	1    0    0    -1
+$EndComp
+$Comp
+L Mechanical:MountingHole H3
+U 1 1 5C846066
+P 3450 8100
+F 0 "H3" H 3550 8146 50  0000 L CNN
+F 1 "MountingHole" H 3750 8800 50  0000 L CNN
+F 2 "sb_designed_footprints:MountingHole_3mm" H 3450 8100 50  0001 C CNN
+F 3 "~" H 3450 8100 50  0001 C CNN
+	1    3450 8100
+	1    0    0    -1
+$EndComp
+$Comp
+L Connector_Generic:Conn_02x06_Counter_Clockwise J6
+U 1 1 5C8539A8
+P 10150 9450
+F 0 "J6" H 10200 9867 50  0000 C CNN
+F 1 "Conn_02x06_Counter_Clockwise" H 10200 9776 50  0000 C CNN
+F 2 "Connector_PinHeader_2.54mm:PinHeader_2x06_P2.54mm_Vertical" H 10150 9450 50  0001 C CNN
+F 3 "~" H 10150 9450 50  0001 C CNN
+	1    10150 9450
+	1    0    0    -1
+$EndComp
+Wire Wire Line
+	10650 8600 10650 9350
+Wire Wire Line
+	10650 9350 10450 9350
+Connection ~ 10650 8600
+Wire Wire Line
+	10650 8600 10450 8600
+Wire Wire Line
+	10550 8500 10550 9250
+Wire Wire Line
+	10550 9250 10450 9250
+Connection ~ 10550 8500
+Wire Wire Line
+	10550 8500 10450 8500
+Wire Wire Line
+	9950 9250 9350 9250
+Wire Wire Line
+	9100 9350 9950 9350
+Wire Wire Line
+	9950 9450 9950 9550
+Wire Wire Line
+	9950 10100 9750 10100
+Connection ~ 9950 9550
+Wire Wire Line
+	9950 9550 9950 9650
+Connection ~ 9950 9650
+Wire Wire Line
+	9950 9650 9950 9750
+Connection ~ 9950 9750
+Wire Wire Line
+	9950 9750 9950 10000
+$Comp
+L power:GND #PWR0107
+U 1 1 5C863787
+P 9350 9250
+F 0 "#PWR0107" H 9350 9000 50  0001 C CNN
+F 1 "GND" V 9355 9122 50  0000 R CNN
+F 2 "" H 9350 9250 50  0001 C CNN
+F 3 "" H 9350 9250 50  0001 C CNN
+	1    9350 9250
+	0    1    -1   0
+$EndComp
+$Comp
+L power:GND #PWR0106
+U 1 1 5C8B7CC6
+P 9750 10100
+F 0 "#PWR0106" H 9750 9850 50  0001 C CNN
+F 1 "GND" V 9755 9972 50  0000 R CNN
+F 2 "" H 9750 10100 50  0001 C CNN
+F 3 "" H 9750 10100 50  0001 C CNN
+	1    9750 10100
+	0    1    -1   0
+$EndComp
+Connection ~ 9950 10000
+Wire Wire Line
+	9950 10000 9950 10100
+Wire Wire Line
+	10450 9650 11700 9650
+Connection ~ 11700 9650
+Wire Wire Line
+	11700 9650 11700 10300
+Wire Wire Line
+	9950 10000 10550 10000
+Wire Wire Line
+	10450 9450 10550 9450
+Wire Wire Line
+	10550 9450 10550 9550
+Wire Wire Line
+	10450 9550 10550 9550
+Connection ~ 10550 9550
+Wire Wire Line
+	10550 9550 10550 9750
+Wire Wire Line
+	10450 9750 10550 9750
+Connection ~ 10550 9750
+Wire Wire Line
+	10550 9750 10550 10000
 $EndSCHEMATC

Commit message: update layout
Connections:
- net +3V3: now also J4.15 (Pin_15), J4.7 (Pin_7); no longer J4.4 (Pin_4)
- net GND: now also J4.16 (Pin_16), J4.8 (Pin_8), J4.9 (Pin_9); no longer J4.11 (Pin_11), J4.3 (Pin_3)
- net at U4.12 (IO27): now also J4.3 (Pin_3); no longer J4.5 (Pin_5)
- net at U4.13 (IO14): now also J4.4 (Pin_4); no longer J4.6 (Pin_6)
- net at U4.14 (IO12): now also J4.5 (Pin_5); no longer J4.7 (Pin_7)
- net at U4.16 (IO13): now also J4.6 (Pin_6); no longer J4.8 (Pin_8)
- net at U4.23 (IO15): no longer J4.16 (Pin_16)
- net at U4.24 (IO2): now also J4.14 (Pin_14); no longer J4.15 (Pin_15)
- net at U4.26 (IO4): now also J4.13 (Pin_13); no longer J4.14 (Pin_14)
- net at J4.12 (Pin_12), J6.11 (Pin_11): now also U4.27 (IO16); no longer U4.28 (IO17)
- new net: J4.11 (Pin_11), J6.12 (Pin_12), U4.28 (IO17)
- no-connect marks 8 -> 7
Changed lines of the file:
@@
 	9500 6950 9500 7700
 Wire Wire Line
-	11700 7300 11700 9650
-Wire Wire Line
 	11000 7700 12500 7700
-Wire Wire Line
-	11300 6250 11300 8400
-Wire Wire Line
-	10450 8700 10750 8700
-Wire Wire Line
-	10450 8800 11150 8800
 $Comp
 L power:+3.3V #PWR0110
 U 1 1 5C79FDEE
-P 11150 8800
-F 0 "#PWR0110" H 11150 8650 50  0001 C CNN
-F 1 "+3.3V" H 11165 8973 50  0000 C CNN
-F 2 "" H 11150 8800 50  0001 C CNN
-F 3 "" H 11150 8800 50  0001 C CNN
-	1    11150 8800
+P 11350 8800
+F 0 "#PWR0110" H 11350 8650 50  0001 C CNN
+F 1 "+3.3V" H 11365 8973 50  0000 C CNN
+F 2 "" H 11350 8800 50  0001 C CNN
+F 3 "" H 11350 8800 50  0001 C CNN
+	1    11350 8800
 	0    1    1    0
 $EndComp
@@
 L power:GND #PWR0111
 U 1 1 5C7A5B81
-P 10750 8700
-F 0 "#PWR0111" H 10750 8450 50  0001 C CNN
-F 1 "GND" V 10755 8572 50  0000 R CNN
-F 2 "" H 10750 8700 50  0001 C CNN
-F 3 "" H 10750 8700 50  0001 C CNN
-	1    10750 8700
+P 11050 8900
+F 0 "#PWR0111" H 11050 8650 50  0001 C CNN
+F 1 "GND" V 11055 8772 50  0000 R CNN
+F 2 "" H 11050 8900 50  0001 C CNN
+F 3 "" H 11050 8900 50  0001 C CNN
+	1    11050 8900
 	0    -1   1    0
 $EndComp
@@
 $EndComp
 $Comp
-L power:GND #PWR0114
-U 1 1 5C897D4A
-P 9450 8400
-F 0 "#PWR0114" H 9450 8150 50  0001 C CNN
-F 1 "GND" V 9455 8272 50  0000 R CNN
-F 2 "" H 9450 8400 50  0001 C CNN
-F 3 "" H 9450 8400 50  0001 C CNN
-	1    9450 8400
-	0    1    -1   0
-$EndComp
-$Comp
 L power:+3.3V #PWR0112
 U 1 1 5C7A5D9B
@@
 	0    -1   -1   0
 $EndComp
-$Comp
-L power:+3.3V #PWR0115
-U 1 1 5C89FA09
-P 9150 8500
-F 0 "#PWR0115" H 9150 8350 50  0001 C CNN
-F 1 "+3.3V" V 9050 8700 50  0000 C CNN
-F 2 "" H 9150 8500 50  0001 C CNN
-F 3 "" H 9150 8500 50  0001 C CNN
-	1    9150 8500
-	0    -1   -1   0
-$EndComp
-NoConn ~ 10450 8900
 Wire Wire Line
 	9150 6300 8500 6300
 Wire Wire Line
-	8500 6300 8500 8600
-Wire Wire Line
-	8550 6400 8550 8700
-Wire Wire Line
-	10450 6950 10450 8200
-Wire Wire Line
-	10550 8300 10450 8300
-Wire Wire Line
-	10550 6950 10550 8300
-Wire Wire Line
-	10450 8400 11300 8400
-Wire Wire Line
-	11200 8500 10550 8500
-Wire Wire Line
-	11200 6150 11200 8500
-Wire Wire Line
-	11250 8600 10650 8600
-Wire Wire Line
-	11250 6050 11250 8600
-Wire Wire Line
-	9450 8200 9950 8200
-Wire Wire Line
-	9150 8300 9950 8300
-Wire Wire Line
-	9450 8400 9950 8400
-Wire Wire Line
-	9150 8500 9950 8500
-Wire Wire Line
-	9750 8900 9950 8900
-Wire Wire Line
-	9750 6950 9750 8900
-Wire Wire Line
-	9950 8800 8600 8800
-Wire Wire Line
-	8600 6500 8600 8800
-Wire Wire Line
-	9950 8700 8550 8700
-Wire Wire Line
-	9950 8600 8500 8600
+	8500 6300 8500 8400
+Wire Wire Line
+	8550 6400 8550 8500
+Wire Wire Line
+	9450 8200 9550 8200
+Wire Wire Line
+	9150 8300 9600 8300
+Wire Wire Line
+	9750 6950 9750 8700
+Wire Wire Line
+	8600 6500 8600 8600
 $Comp
 L Mechanical:MountingHole H2
@@
 $EndComp
 Wire Wire Line
-	10650 8600 10650 9350
-Wire Wire Line
-	10650 9350 10450 9350
-Connection ~ 10650 8600
-Wire Wire Line
-	10650 8600 10450 8600
-Wire Wire Line
-	10550 8500 10550 9250
-Wire Wire Line
-	10550 9250 10450 9250
-Connection ~ 10550 8500
-Wire Wire Line
-	10550 8500 10450 8500
-Wire Wire Line
 	9950 9250 9350 9250
 Wire Wire Line
 	9100 9350 9950 9350
-Wire Wire Line
-	9950 9450 9950 9550
-Wire Wire Line
-	9950 10100 9750 10100
-Connection ~ 9950 9550
-Wire Wire Line
-	9950 9550 9950 9650
-Connection ~ 9950 9650
-Wire Wire Line
-	9950 9650 9950 9750
-Connection ~ 9950 9750
-Wire Wire Line
-	9950 9750 9950 10000
 $Comp
 L power:GND #PWR0107
@@
 	0    1    -1   0
 $EndComp
+Wire Wire Line
+	10450 9450 10550 9450
+Wire Wire Line
+	10450 9550 10550 9550
+Wire Wire Line
+	9950 10100 9750 10100
+Wire Wire Line
+	10450 9750 10550 9750
+Wire Wire Line
+	9950 9550 9950 9650
+Connection ~ 9950 9550
+Wire Wire Line
+	9950 9450 9950 9550
+Connection ~ 9950 9650
+Wire Wire Line
+	9950 9650 9950 9750
+Connection ~ 9950 9750
+Wire Wire Line
+	10550 9550 10550 9750
+Connection ~ 10550 9550
+Wire Wire Line
+	10550 9450 10550 9550
+Connection ~ 10550 9750
+Wire Wire Line
+	10550 9750 10550 10000
+Wire Wire Line
+	11700 7300 11700 9650
+Wire Wire Line
+	11700 9650 11700 10300
+Connection ~ 11700 9650
+Wire Wire Line
+	10450 9650 11700 9650
+Wire Wire Line
+	9950 10000 9950 10100
+Wire Wire Line
+	9950 9750 9950 10000
 Connection ~ 9950 10000
 Wire Wire Line
-	9950 10000 9950 10100
-Wire Wire Line
-	10450 9650 11700 9650
-Connection ~ 11700 9650
-Wire Wire Line
-	11700 9650 11700 10300
-Wire Wire Line
 	9950 10000 10550 10000
 Wire Wire Line
-	10450 9450 10550 9450
-Wire Wire Line
-	10550 9450 10550 9550
-Wire Wire Line
-	10450 9550 10550 9550
-Connection ~ 10550 9550
-Wire Wire Line
-	10550 9550 10550 9750
-Wire Wire Line
-	10450 9750 10550 9750
-Connection ~ 10550 9750
-Wire Wire Line
-	10550 9750 10550 10000
+	9950 8400 8500 8400
+Wire Wire Line
+	9950 8500 8550 8500
+Wire Wire Line
+	9950 8600 8600 8600
+Wire Wire Line
+	9750 8700 9950 8700
+Wire Wire Line
+	9550 8900 9550 8200
+Wire Wire Line
+	9550 8900 9950 8900
+Connection ~ 9550 8200
+Wire Wire Line
+	9550 8200 9950 8200
+Wire Wire Line
+	9950 8800 9600 8800
+Wire Wire Line
+	9600 8800 9600 8300
+Connection ~ 9600 8300
+Wire Wire Line
+	9600 8300 9950 8300
+Wire Wire Line
+	10450 8900 10750 8900
+Wire Wire Line
+	11350 8800 10650 8800
+Wire Wire Line
+	10550 8400 10450 8400
+Wire Wire Line
+	10550 6950 10550 8400
+Wire Wire Line
+	10450 8300 10650 8300
+Wire Wire Line
+	10650 8300 10650 8800
+Connection ~ 10650 8800
+Wire Wire Line
+	10650 8800 10450 8800
+Wire Wire Line
+	10450 8200 10750 8200
+Wire Wire Line
+	10750 8200 10750 8900
+Connection ~ 10750 8900
+Wire Wire Line
+	10750 8900 11050 8900
+Wire Wire Line
+	11300 6250 11300 8500
+Wire Wire Line
+	10450 8700 10850 8700
+Wire Wire Line
+	11250 6050 11250 8700
+Wire Wire Line
+	10450 8600 10950 8600
+Wire Wire Line
+	11200 6150 11200 8600
+Wire Wire Line
+	10450 8500 11300 8500
+Wire Wire Line
+	10850 8700 10850 9250
+Wire Wire Line
+	10450 9250 10850 9250
+Connection ~ 10850 8700
+Wire Wire Line
+	10850 8700 11250 8700
+Wire Wire Line
+	10950 8600 10950 9350
+Wire Wire Line
+	10450 9350 10950 9350
+Connection ~ 10950 8600
+Wire Wire Line
+	10950 8600 11200 8600
 $EndSCHEMATC

Commit message: redesign
Parts:
- added D1: LED_Small, LED_SMD:LED_0603_1608Metric_Pad1.05x0.95mm_HandSolder, symbol Device:LED_Small
- added R1: R_Small, Resistor_SMD:R_0603_1608Metric, symbol Device:R_Small
Connections:
- net GND: now also D1.1 (K)
- net at U4.23 (IO15): now also R1.2
- new net: D1.2 (A), R1.1
Changed lines of the file:
@@
 $EndComp
 Wire Wire Line
-	13050 6650 13350 6650
+	13050 6650 13150 6650
 $Comp
 L power:GND #PWR0103
@@
 	9150 8300 9600 8300
 Wire Wire Line
-	9750 6950 9750 8700
-Wire Wire Line
 	8600 6500 8600 8600
 $Comp
@@
 	9950 8600 8600 8600
 Wire Wire Line
-	9750 8700 9950 8700
-Wire Wire Line
 	9550 8900 9550 8200
 Wire Wire Line
@@
 Wire Wire Line
 	10950 8600 11200 8600
+Wire Wire Line
+	9750 8700 9950 8700
+Wire Wire Line
+	9750 6950 9750 8700
+$Comp
+L Device:LED_Small D1
+U 1 1 5C9D26F7
+P 12400 7500
+F 0 "D1" H 12400 7295 50  0000 C CNN
+F 1 "LED_Small" H 12400 7386 50  0000 C CNN
+F 2 "LED_SMD:LED_0603_1608Metric_Pad1.05x0.95mm_HandSolder" V 12400 7500 50  0001 C CNN
+F 3 "~" V 12400 7500 50  0001 C CNN
+	1    12400 7500
+	-1   0    0    1
+$EndComp
+$Comp
+L Device:R_Small R1
+U 1 1 5C9DFC41
+P 11950 7500
+F 0 "R1" V 11754 7500 50  0000 C CNN
+F 1 "R_Small" V 11845 7500 50  0000 C CNN
+F 2 "Resistor_SMD:R_0603_1608Metric" H 11950 7500 50  0001 C CNN
+F 3 "~" H 11950 7500 50  0001 C CNN
+	1    11950 7500
+	0    1    1    0
+$EndComp
+Wire Wire Line
+	11850 7500 10450 7500
+Wire Wire Line
+	10450 7500 10450 6950
+Wire Wire Line
+	12050 7500 12300 7500
+Wire Wire Line
+	13150 6650 13150 7500
+Wire Wire Line
+	12500 7500 13150 7500
+Connection ~ 13150 6650
+Wire Wire Line
+	13150 6650 13350 6650
 $EndSCHEMATC
