File: portia.kicad_pcb (KiCad board)
At the start: 2 copper layers, 42.5 x 31 mm, 13 parts, among them J1 Conn_01x11, J2 Conn_01x11, J4 Conn_02x06_Odd_Even, SW1 Reset, SW2 Reset, U1 LM1117-3.3, U4 ESP32-WROOM

Commit message: update layout
Parts:
- removed C1, C2: C_Small, Capacitor_SMD:C_0603_1608Metric_Pad1.05x0.95mm_HandSolder
- removed U1: LM1117-3.3, Package_TO_SOT_SMD:SOT-223
- added J3: Conn_01x02, Connector_PinHeader_2.54mm:PinHeader_1x02_P2.54mm_Vertical, F.Cu at (159.0, 111.3)
- added J5: Conn_01x08, Connector_PinHeader_2.54mm:PinHeader_1x08_P2.54mm_Vertical, F.Cu at (196.5, 132.3)
- H1, H5: footprint MountingHole:MountingHole_3mm -> sb_designed_footprints:MountingHole_3mm
- J1: value Conn_01x11 -> Conn_01x02; footprint Connector_PinHeader_2.54mm:PinHeader_1x11_P2.54mm_Vertical -> Connector_PinHeader_2.54mm:PinHeader_1x02_P2.54mm_Vertical
- J2: value Conn_01x11 -> Conn_01x08; footprint Connector_PinHeader_2.54mm:PinHeader_1x11_P2.54mm_Vertical -> Connector_PinHeader_2.54mm:PinHeader_1x08_P2.54mm_Vertical
- J4: value Conn_02x06_Odd_Even -> Conn_02x08_Counter_Clockwise
- moved J2 32.0 mm to (178.8, 105.3), turned to 90 degrees
- moved J1 23.6 mm to (158.7, 125.8)
- moved J4 6.41 mm to (173.5, 117.0), turned to 0 degrees
- moved R6 3.37 mm to (165.8, 105.8), turned to 270 degrees
- moved SW1 3.27 mm to (169.5, 105.8)
- moved SW2 2.78 mm to (169.0, 131.3)
- moved R4 2.47 mm to (164.8, 131.3), turned to 90 degrees
Connections:
- J1 pad 1: Net-(J1-Pad1) -> +3V3
- J1 pad 2: Net-(J1-Pad2) -> GND
- J2 pad 1: GND -> Net-(J2-Pad1)
- J2 pad 2: GND -> Net-(J2-Pad2)
- J2 pad 3: +3V3 -> Net-(J2-Pad3)
- J4 pad 1: Net-(J4-Pad1) -> GND
- J4 pad 10: GND -> +3V3
- J4 pad 11: +3V3 -> GND
- J4 pad 12: +3V3 -> Net-(J4-Pad12)
- J4 pad 2: Net-(J4-Pad2) -> +3V3
- J4 pad 3: Net-(J4-Pad3) -> GND
- J4 pad 4: Net-(J4-Pad4) -> +3V3
- J4 pad 9: GND -> Net-(J4-Pad9)
- U4 pad 10: Net-(J1-Pad2) -> Net-(J2-Pad2)
- U4 pad 11: Net-(J1-Pad1) -> Net-(J2-Pad1)
- U4 pad 13: Net-(J4-Pad3) -> Net-(J4-Pad6)
- U4 pad 14: Net-(J4-Pad1) -> Net-(J4-Pad7)
- U4 pad 16: Net-(J4-Pad7) -> Net-(J4-Pad8)
- U4 pad 23: Net-(U4-Pad23) -> Net-(J4-Pad16)
- U4 pad 24: Net-(J4-Pad8) -> Net-(J4-Pad15)
- U4 pad 26: Net-(J4-Pad6) -> Net-(J4-Pad14)
- U4 pad 27: Net-(J4-Pad2) -> Net-(J4-Pad13)
- U4 pad 28: Net-(J4-Pad4) -> Net-(J4-Pad12)
- U4 pad 29: Net-(J2-Pad11) -> Net-(J5-Pad8)
- U4 pad 30: Net-(J2-Pad10) -> Net-(J5-Pad7)
- U4 pad 31: Net-(J2-Pad9) -> Net-(J5-Pad6)
- U4 pad 33: Net-(J2-Pad8) -> Net-(J5-Pad5)
- U4 pad 34: Net-(J2-Pad7) -> Net-(J5-Pad4)
- U4 pad 35: Net-(J2-Pad6) -> Net-(J5-Pad3)
- U4 pad 36: Net-(J2-Pad5) -> Net-(J5-Pad2)
- U4 pad 37: Net-(J2-Pad4) -> Net-(J5-Pad1)
- U4 pad 4: Net-(J1-Pad8) -> Net-(J2-Pad8)
- U4 pad 5: Net-(J1-Pad7) -> Net-(J2-Pad7)
- U4 pad 6: Net-(J1-Pad6) -> Net-(J2-Pad6)
- U4 pad 7: Net-(J1-Pad5) -> Net-(J2-Pad5)
- U4 pad 8: Net-(J1-Pad4) -> Net-(J2-Pad4)
- U4 pad 9: Net-(J1-Pad3) -> Net-(J2-Pad3)
Routing:
- net Net-(J1-Pad1): track 17.0 -> 0.00 mm
- net Net-(J1-Pad2): track 14.8 -> 0.00 mm
- net Net-(J1-Pad3): track 14.3 -> 0.00 mm, vias 1 -> 0
- net Net-(J1-Pad4): track 13.0 -> 0.00 mm, vias 1 -> 0
- net Net-(J1-Pad5): track 11.8 -> 0.00 mm, vias 1 -> 0
- net Net-(J2-Pad6): track 12.3 -> 0.63 mm
- net Net-(J2-Pad5): track 11.3 -> 0.00 mm
- net Net-(J1-Pad6): track 10.4 -> 0.00 mm
- net Net-(J2-Pad4): track 10.3 -> 0.00 mm
- net Net-(J1-Pad7): track 9.62 -> 0.00 mm
- net Net-(J1-Pad8): track 7.19 -> 0.00 mm
- net Net-(R6-Pad1): track 2.00 -> 0.00 mm, vias 1 -> 0
- net Net-(J2-Pad7): track 0.00 -> 0.80 mm
Other:
- board size 42.5 x 31 mm -> 49 x 31 mm
