File: portia.kicad_pcb (KiCad board)
At the start: 2 copper layers, 49 x 31 mm, 12 parts, among them J1 Conn_01x02, J2 Conn_01x08, J3 Conn_01x02, J4 Conn_02x08_Counter_Clockwise, J5 Conn_01x08, SW1 Reset, SW2 Reset, U4 ESP32-WROOM

Commit message: update layout
Parts:
- removed J1, J3: Conn_01x02, Connector_PinHeader_2.54mm:PinHeader_1x02_P2.54mm_Vertical
- removed SW1, SW2: Reset, Button_Switch_SMD:SW_SPST_B3U-1000P-B
- added Boot: Boot_ESP, Button_Switch_SMD:SW_SPST_B3U-1000P-B, F.Cu at (171.0, 131.9)
- added H2: MountingHole, sb_designed_footprints:MountingHole_3mm, F.Cu at (202.0, 107.3)
- added H3: MountingHole, sb_designed_footprints:MountingHole_3mm, F.Cu at (202.0, 130.3)
- added J6: Conn_02x06_Counter_Clockwise, Connector_PinHeader_2.54mm:PinHeader_2x06_P2.54mm_Vertical, F.Cu at (159.0, 113.3)
- added Reset: EN, Button_Switch_SMD:SW_SPST_B3U-1000P-B, F.Cu at (171.0, 105.8)
- moved R4 10.0 mm to (174.8, 131.8), turned to 270 degrees
- moved R6 8.97 mm to (174.7, 105.5), turned to 90 degrees
Routing:
- net Net-(J4-Pad12): track 0.00 -> 31.9 mm, vias 0 -> 1
- net Net-(R6-Pad1): track 0.00 -> 30.8 mm, vias 0 -> 2
- net Net-(J4-Pad13): track 0.00 -> 27.2 mm, vias 0 -> 1
- net Net-(J4-Pad5): track 0.00 -> 16.6 mm
- net Net-(J4-Pad14): track 0.00 -> 14.8 mm
- net Net-(J4-Pad6): track 0.00 -> 13.4 mm
- net +3V3: track 0.00 -> 13.2 mm, vias 0 -> 6
- net Net-(Boot1-Pad1): track 0.00 -> 11.1 mm, vias 0 -> 2
- net Net-(J4-Pad15): track 0.00 -> 9.94 mm
- net Net-(J5-Pad8): track 0.00 -> 9.87 mm
- net Net-(J4-Pad7): track 0.00 -> 9.25 mm
- net Net-(J2-Pad1): track 0.00 -> 9.15 mm
- net Net-(J5-Pad7): track 0.00 -> 8.71 mm
- net Net-(J5-Pad5): track 0.00 -> 7.55 mm
- net Net-(J5-Pad6): track 0.00 -> 7.40 mm
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- added copper zone on B.Cu, net +3V3
- added copper zone on F.Cu, net GND
Other:
- board size 49 x 31 mm -> 50 x 31 mm
- board text added: "18"
- board text added: "19"
- board text added: "21"
- board text added: "22"
- board text added: "23"
- board text added: "25"
- board text added: "26"
- board text added: "3.3"
- board text added: "32"
- board text added: "33"
- board text added: "34"
- board text added: "35"
- board text added: "5"
- board text added: "gnd"
- board text added: "rx"
- board text added: "tx"
- board text added: "vn"
- board text added: "vp"

Commit message: update layout
Parts:
- removed Boot: Boot_ESP, Button_Switch_SMD:SW_SPST_B3U-1000P-B
- removed Reset: EN, Button_Switch_SMD:SW_SPST_B3U-1000P-B
- added Boot1: Boot_ESP, Button_Switch_SMD:SW_SPST_B3U-1000P-B, F.Cu at (166.0, 142.7)
- added Reset1: EN, Button_Switch_SMD:SW_SPST_B3U-1000P-B, F.Cu at (175.9, 143.4)
Connections:
- J4 pad 11: GND -> Net-(J4-Pad11)
- J4 pad 15: Net-(J4-Pad15) -> +3V3
- J4 pad 16: Net-(J4-Pad16) -> GND
- J4 pad 3: GND -> Net-(J4-Pad3)
- J4 pad 4: +3V3 -> Net-(J4-Pad4)
- J4 pad 7: Net-(J4-Pad7) -> +3V3
- J4 pad 8: Net-(J4-Pad8) -> GND
- J4 pad 9: Net-(J4-Pad9) -> GND
- J6 pad 11: Net-(J4-Pad12) -> Net-(J6-Pad11)
- J6 pad 12: Net-(J4-Pad13) -> Net-(J6-Pad12)
- U4 pad 12: Net-(J4-Pad5) -> Net-(J4-Pad3)
- U4 pad 13: Net-(J4-Pad6) -> Net-(J4-Pad4)
- U4 pad 14: Net-(J4-Pad7) -> Net-(J4-Pad5)
- U4 pad 16: Net-(J4-Pad8) -> Net-(J4-Pad6)
- U4 pad 23: Net-(J4-Pad16) -> Net-(U4-Pad23)
- U4 pad 24: Net-(J4-Pad15) -> Net-(J4-Pad14)
- U4 pad 26: Net-(J4-Pad14) -> Net-(J4-Pad13)
- U4 pad 27: Net-(J4-Pad13) -> Net-(J4-Pad12)
- U4 pad 28: Net-(J4-Pad12) -> Net-(J4-Pad11)
Routing:
- net Net-(J4-Pad3): track 0.00 -> 20.0 mm
- net Net-(J4-Pad11): track 0.00 -> 19.5 mm, vias 0 -> 1
- net Net-(J4-Pad4): track 0.00 -> 16.5 mm
- net Net-(J4-Pad12): track 31.9 -> 16.7 mm
- net Net-(J4-Pad6): track 13.4 -> 0.00 mm
- net Net-(J4-Pad13): track 27.2 -> 16.3 mm, vias 1 -> 0
- net Net-(J4-Pad15): track 9.94 -> 0.00 mm
- net Net-(J4-Pad7): track 9.25 -> 0.00 mm
- net Net-(J4-Pad16): track 6.46 -> 0.00 mm
- net Net-(J4-Pad8): track 6.40 -> 0.00 mm
- net Net-(J4-Pad5): track 16.6 -> 12.2 mm
- net Net-(J4-Pad14): track 14.8 -> 11.3 mm
- net Net-(J6-Pad11): track 0.00 -> 3.19 mm
- net Net-(J6-Pad12): track 0.00 -> 2.13 mm

Commit message: redesign
Parts:
- added D1: LED_Small, LED_SMD:LED_0603_1608Metric_Pad1.05x0.95mm_HandSolder, F.Cu at (164.0, 129.9)
- added R1: R_Small, Resistor_SMD:R_0603_1608Metric, F.Cu at (164.8, 133.2)
- moved Reset1 39.1 mm to (165.2, 105.7), turned to 180 degrees
- moved Boot1 11.2 mm to (170.2, 132.2), turned to 180 degrees
Connections:
- J6 pad 11: Net-(J6-Pad11) -> Net-(J4-Pad12)
- J6 pad 12: Net-(J6-Pad12) -> Net-(J4-Pad11)
Routing:
- net Net-(R1-Pad2): track 0.00 -> 21.4 mm, vias 0 -> 2
- net Net-(J4-Pad12): track 16.7 -> 32.2 mm
- net Net-(J4-Pad6): track 0.00 -> 14.2 mm, vias 0 -> 2
- net Net-(J4-Pad11): track 19.5 -> 30.8 mm
- net Net-(R6-Pad1): track 30.8 -> 38.2 mm
- net Net-(J6-Pad11): track 3.19 -> 0.00 mm
- net Net-(D1-Pad2): track 0.00 -> 2.39 mm
- net Net-(J6-Pad12): track 2.13 -> 0.00 mm
- net +3V3: track 12.7 -> 14.7 mm, vias 6 -> 7
- net Net-(Boot1-Pad1): track 11.1 -> 11.8 mm
- net Net-(J4-Pad13): track 16.3 -> 16.9 mm

Commit message: update design
Connections:
- J6 pad 1: GND -> Net-(J4-Pad4)
- J6 pad 2: +3V3 -> Net-(J4-Pad3)
- J6 pad 3: GND -> Net-(J4-Pad6)
- J6 pad 4: GND -> Net-(J4-Pad5)
- U4 pad 12: Net-(J4-Pad3) -> Net-(U4-Pad12)
- U4 pad 13: Net-(J4-Pad4) -> Net-(U4-Pad13)
- U4 pad 14: Net-(J4-Pad5) -> Net-(U4-Pad14)
- U4 pad 16: Net-(J4-Pad6) -> Net-(U4-Pad16)
Routing:
- net Net-(J4-Pad6): track 14.2 -> 25.4 mm, vias 2 -> 1
- net Net-(J4-Pad3): track 20.0 -> 12.4 mm
- net Net-(J4-Pad5): track 12.5 -> 18.0 mm, vias 0 -> 1
- net Net-(J4-Pad4): track 16.5 -> 15.3 mm
- net Net-(U4-Pad13): track 0.00 -> 1.12 mm
Changed lines of the file:
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@@
   (general
     (thickness 1.6)
-    (drawings 41)
-    (tracks 190)
+    (drawings 37)
+    (tracks 193)
     (zones 0)
     (modules 15)
-    (nets 38)
+    (nets 42)
   )
   (page A4)
@@
     (solder_mask_min_width 0.25)
     (aux_axis_origin 160.02 107.28)
-    (grid_origin 165.5675 133.169)
+    (grid_origin 174.76 111.259)
     (visible_elements FFFFF77F)
     (pcbplotparams
@@
   (net 36 "Net-(D1-Pad2)")
   (net 37 "Net-(R1-Pad2)")
+  (net 38 "Net-(U4-Pad16)")
+  (net 39 "Net-(U4-Pad14)")
+  (net 40 "Net-(U4-Pad13)")
+  (net 41 "Net-(U4-Pad12)")
   (net_class Default "This is the default net class."
     (clearance 0.2)
@@
     (add_net "Net-(R1-Pad2)")
     (add_net "Net-(R6-Pad1)")
+    (add_net "Net-(U4-Pad12)")
+    (add_net "Net-(U4-Pad13)")
+    (add_net "Net-(U4-Pad14)")
+    (add_net "Net-(U4-Pad16)")
     (add_net "Net-(U4-Pad17)")
     (add_net "Net-(U4-Pad18)")
@@
     )
     (pad 1 thru_hole circle (at 0 0) (size 1.7 1.7) (drill 1) (layers *.Cu *.Mask)
-      (net 2 GND))
+      (net 34 "Net-(J4-Pad4)"))
     (pad 2 thru_hole oval (at 2.54 0) (size 1.7 1.7) (drill 1) (layers *.Cu *.Mask)
-      (net 1 +3V3))
+      (net 33 "Net-(J4-Pad3)"))
     (pad 3 thru_hole oval (at 0 2.54) (size 1.7 1.7) (drill 1) (layers *.Cu *.Mask)
-      (net 2 GND))
+      (net 17 "Net-(J4-Pad6)"))
     (pad 4 thru_hole oval (at 2.54 2.54) (size 1.7 1.7) (drill 1) (layers *.Cu *.Mask)
-      (net 2 GND))
+      (net 16 "Net-(J4-Pad5)"))
     (pad 5 thru_hole oval (at 0 5.08) (size 1.7 1.7) (drill 1) (layers *.Cu *.Mask)
       (net 2 GND))
@@
       (net 9 "Net-(U4-Pad17)"))
     (pad 16 smd oval (at 4.445 -12.75 90) (size 0.9 2.5) (layers F.Cu F.Paste F.Mask)
-      (net 17 "Net-(J4-Pad6)"))
+      (net 38 "Net-(U4-Pad16)"))
     (pad 15 smd oval (at 5.715 -12.75 90) (size 0.9 2.5) (layers F.Cu F.Paste F.Mask)
       (net 2 GND))
     (pad 14 smd oval (at 9 -11.26 90) (size 2.5 0.9) (layers F.Cu F.Paste F.Mask)
-      (net 16 "Net-(J4-Pad5)"))
+      (net 39 "Net-(U4-Pad14)"))
     (pad 13 smd oval (at 9 -9.99 90) (size 2.5 0.9) (layers F.Cu F.Paste F.Mask)
-      (net 34 "Net-(J4-Pad4)"))
+      (net 40 "Net-(U4-Pad13)"))
     (pad 12 smd oval (at 9 -8.72 90) (size 2.5 0.9) (layers F.Cu F.Paste F.Mask)
-      (net 33 "Net-(J4-Pad3)"))
+      (net 41 "Net-(U4-Pad12)"))
     (pad 11 smd oval (at 9 -7.45 90) (size 2.5 0.9) (layers F.Cu F.Paste F.Mask)
       (net 28 "Net-(J2-Pad1)"))
@@
     (effects (font (size 0.5 0.5) (thickness 0.125)))
   )
-  (gr_text "gnd\n" (at 163.42 115.88 90) (layer F.SilkS)
-    (effects (font (size 0.5 0.5) (thickness 0.125)))
-  )
-  (gr_text "3.3\n" (at 163.42 113.48 90) (layer F.SilkS)
-    (effects (font (size 0.5 0.5) (thickness 0.125)))
-  )
   (gr_text "gnd\n" (at 157.02 123.48 90) (layer F.SilkS)
     (effects (font (size 0.5 0.5) (thickness 0.125)))
@@
   )
   (gr_text "gnd\n" (at 157.02 118.48 90) (layer F.SilkS)
-    (effects (font (size 0.5 0.5) (thickness 0.125)))
-  )
-  (gr_text "gnd\n" (at 157.02 115.88 90) (layer F.SilkS)
-    (effects (font (size 0.5 0.5) (thickness 0.125)))
-  )
-  (gr_text "gnd\n" (at 157.02 113.28 90) (layer F.SilkS)
     (effects (font (size 0.5 0.5) (thickness 0.125)))
   )
@@
   (segment (start 193.69 106.6965) (end 194.6035 106.6965) (width 0.25) (layer F.Cu) (net 15))
   (segment (start 194.6035 106.6965) (end 196.02 105.28) (width 0.25) (layer F.Cu) (net 15))
-  (segment (start 170.95 109.184) (end 170.95 111.259) (width 0.25) (layer F.Cu) (net 16))
-  (segment (start 180.52 109.724) (end 179.82 109.724) (width 0.25) (layer F.Cu) (net 16))
-  (segment (start 179.82 109.724) (end 178.57 108.474) (width 0.25) (layer F.Cu) (net 16))
-  (segment (start 171.66 108.474) (end 170.95 109.184) (width 0.25) (layer F.Cu) (net 16))
-  (segment (start 178.57 108.474) (end 171.66 108.474) (width 0.25) (layer F.Cu) (net 16))
-  (segment (start 172.22 111.259) (end 172.22 109.259) (width 0.25) (layer F.Cu) (net 17))
-  (segment (start 172.22 109.259) (end 172.22 109.259) (width 0.25) (layer F.Cu) (net 17))
-  (via (at 172.22 109.259) (size 0.6) (drill 0.4) (layers F.Cu B.Cu) (net 17))
-  (segment (start 179.03 114.279) (end 176.78 114.279) (width 0.25) (layer F.Cu) (net 17))
-  (segment (start 176.78 114.279) (end 176.78 114.279) (width 0.25) (layer F.Cu) (net 17))
-  (via (at 176.78 114.279) (size 0.6) (drill 0.4) (layers F.Cu B.Cu) (net 17))
-  (segment (start 172.519999 108.959001) (end 172.22 109.259) (width 0.25) (layer B.Cu) (net 17))
-  (segment (start 176.78 114.279) (end 176.78 110.029) (width 0.25) (layer B.Cu) (net 17))
-  (segment (start 176.78 110.029) (end 175.03 108.279) (width 0.25) (layer B.Cu) (net 17))
-  (segment (start 175.03 108.279) (end 173.2 108.279) (width 0.25) (layer B.Cu) (net 17))
-  (segment (start 173.2 108.279) (end 172.519999 108.959001) (width 0.25) (layer B.Cu) (net 17))
+  (segment (start 170.95 111.259) (end 170.95 107.759) (width 0.25) (layer F.Cu) (net 16))
+  (segment (start 170.95 107.759) (end 170.95 107.759) (width 0.25) (layer F.Cu) (net 16))
+  (via (at 170.95 107.759) (size 0.6) (drill 0.4) (layers F.Cu B.Cu) (net 16))
+  (segment (start 163.7 113.764) (end 163.7 110.759) (width 0.25) (layer B.Cu) (net 16))
+  (segment (start 161.58 115.884) (end 163.7 113.764) (width 0.25) (layer B.Cu) (net 16))
+  (segment (start 166.7 107.759) (end 170.95 107.759) (width 0.25) (layer B.Cu) (net 16))
+  (segment (start 163.7 110.759) (end 166.7 107.759) (width 0.25) (layer B.Cu) (net 16))
+  (via (at 172.22 108.509) (size 0.6) (drill 0.4) (layers F.Cu B.Cu) (net 17))
+  (segment (start 172.22 111.259) (end 172.22 108.509) (width 0.25) (layer F.Cu) (net 17))
+  (segment (start 161.2 110.509) (end 164.575001 107.133999) (width 0.25) (layer B.Cu) (net 17))
+  (segment (start 159.04 115.884) (end 157.2 114.044) (width 0.25) (layer B.Cu) (net 17))
+  (segment (start 171.824999 107.133999) (end 172.22 107.529) (width 0.25) (layer B.Cu) (net 17))
+  (segment (start 157.2 112.259) (end 158.95 110.509) (width 0.25) (layer B.Cu) (net 17))
+  (segment (start 164.575001 107.133999) (end 171.824999 107.133999) (width 0.25) (layer B.Cu) (net 17))
+  (segment (start 157.2 114.044) (end 157.2 112.259) (width 0.25) (layer B.Cu) (net 17))
+  (segment (start 172.22 107.529) (end 172.22 108.509) (width 0.25) (layer B.Cu) (net 17))
+  (segment (start 158.95 110.509) (end 161.2 110.509) (width 0.25) (layer B.Cu) (net 17))
   (segment (start 195.76 130.049) (end 195.76 127.724) (width 0.25) (layer F.Cu) (net 18))
   (segment (start 196.52 130.809) (end 195.76 130.049) (width 0.25) (layer F.Cu) (net 18))
@@
   (segment (start 172.185 132.549) (end 171.86 132.224) (width 0.25) (layer F.Cu) (net 32))
   (segment (start 174.76 132.549) (end 172.185 132.549) (width 0.25) (layer F.Cu) (net 32))
-  (segment (start 168.41 108.474) (end 168.41 111.259) (width 0.25) (layer F.Cu) (net 33))
-  (segment (start 169.40399 107.48001) (end 168.41 108.474) (width 0.25) (layer F.Cu) (net 33))
-  (segment (start 182.91601 107.48001) (end 169.40399 107.48001) (width 0.25) (layer F.Cu) (net 33))
-  (segment (start 183.06 109.724) (end 183.06 107.624) (width 0.25) (layer F.Cu) (net 33))
-  (segment (start 183.06 107.624) (end 182.91601 107.48001) (width 0.25) (layer F.Cu) (net 33))
-  (segment (start 169.68 108.454) (end 169.68 111.259) (width 0.25) (layer F.Cu) (net 34))
-  (segment (start 181.79 109.724) (end 181.79 108.604) (width 0.25) (layer F.Cu) (net 34))
-  (segment (start 181.16 107.974) (end 170.16 107.974) (width 0.25) (layer F.Cu) (net 34))
-  (segment (start 181.79 108.604) (end 181.16 107.974) (width 0.25) (layer F.Cu) (net 34))
-  (segment (start 170.16 107.974) (end 169.68 108.454) (width 0.25) (layer F.Cu) (net 34))
+  (segment (start 161.58 113.344) (end 161.58 111.6565) (width 0.25) (layer F.Cu) (net 33))
+  (segment (start 168.41 109.759) (end 168.41 111.259) (width 0.25) (layer F.Cu) (net 33))
+  (segment (start 167.440001 108.233999) (end 168.41 109.203998) (width 0.25) (layer F.Cu) (net 33))
+  (segment (start 168.41 109.203998) (end 168.41 109.759) (width 0.25) (layer F.Cu) (net 33))
+  (segment (start 165.002501 108.233999) (end 167.440001 108.233999) (width 0.25) (layer F.Cu) (net 33))
+  (segment (start 161.58 111.6565) (end 165.002501 108.233999) (width 0.25) (layer F.Cu) (net 33))
+  (segment (start 164.600011 107.783989) (end 159.889999 112.494001) (width 0.25) (layer F.Cu) (net 34))
+  (segment (start 159.889999 112.494001) (end 159.04 113.344) (width 0.25) (layer F.Cu) (net 34))
+  (segment (start 167.704989 107.783989) (end 164.600011 107.783989) (width 0.25) (layer F.Cu) (net 34))
+  (segment (start 169.68 109.759) (end 167.704989 107.783989) (width 0.25) (layer F.Cu) (net 34))
+  (segment (start 169.68 111.259) (end 169.68 109.759) (width 0.25) (layer F.Cu) (net 34))
+  (segment (start 181.79 109.724) (end 181.79 108.604) (width 0.25) (layer F.Cu) (net 40))
   (segment (start 168.41 125.974) (end 168.41 128.724) (width 0.25) (layer F.Cu) (net 35))
   (segment (start 168.41 128.724) (end 168.41 129.474) (width 0.25) (layer F.Cu) (net 35))

Commit message: update redesign
Parts:
- removed D1: LED_Small, LED_SMD:LED_0603_1608Metric_Pad1.05x0.95mm_HandSolder
- removed H3: MountingHole, sb_designed_footprints:MountingHole_3mm
- removed J2, J5: Conn_01x08, Connector_PinHeader_2.54mm:PinHeader_1x08_P2.54mm_Vertical
- removed J4: Conn_02x08_Counter_Clockwise, sb_designed_footprints:castellated12
- removed J6: Conn_02x06_Counter_Clockwise, Connector_PinHeader_2.54mm:PinHeader_2x06_P2.54mm_Vertical
- removed R1: R_Small, Resistor_SMD:R_0603_1608Metric
- moved H5 23.0 mm to (183.0, 130.3)
- moved Reset1 19.5 mm to (180.0, 118.3)
- moved H2 19.0 mm to (183.0, 107.3)
- moved Boot1 13.3 mm to (180.0, 123.3)
- moved U4 7.26 mm to (199.0, 119.3)
- moved R4 6.71 mm to (173.0, 125.3)
Routing:
- net Net-(R6-Pad1): track 38.2 -> 0.00 mm, vias 2 -> 0
- net Net-(J4-Pad12): track 32.2 -> 0.00 mm, vias 1 -> 0
- net Net-(J4-Pad11): track 30.8 -> 0.00 mm, vias 1 -> 0
- net Net-(J4-Pad6): track 25.4 -> 0.00 mm, vias 1 -> 0
- net Net-(R1-Pad2): track 21.4 -> 0.00 mm, vias 2 -> 0
- net Net-(J4-Pad5): track 18.0 -> 0.00 mm, vias 1 -> 0
- net Net-(J4-Pad13): track 16.9 -> 0.00 mm
- net Net-(J4-Pad4): track 15.3 -> 0.00 mm
- net +3V3: track 14.7 -> 0.00 mm, vias 7 -> 0
- net Net-(J4-Pad3): track 12.4 -> 0.00 mm
- net Net-(Boot1-Pad1): track 11.8 -> 0.00 mm, vias 2 -> 0
- net Net-(J4-Pad14): track 11.3 -> 0.00 mm
- net Net-(J5-Pad8): track 9.87 -> 0.00 mm
- net Net-(J2-Pad1): track 9.15 -> 0.00 mm
- net Net-(J5-Pad7): track 8.71 -> 0.00 mm
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Other:
- board text removed: "34"

Commit message: update layout
Parts:
- added C1: 10uf, Capacitor_SMD:C_0603_1608Metric_Pad1.05x0.95mm_HandSolder, F.Cu at (174.5, 105.7)
- added C2: 10uf, Capacitor_SMD:C_0603_1608Metric_Pad1.05x0.95mm_HandSolder, F.Cu at (174.5, 109.7)
- added D1: LED_Small, LED_SMD:LED_0603_1608Metric, F.Cu at (174.0, 113.5)
- added J1: VCC, Connector_PinHeader_2.54mm:PinHeader_1x02_P2.54mm_Vertical, F.Cu at (177.8, 109.0)
- added J2: Conn_01x08, Connector_PinSocket_2.54mm:PinSocket_1x08_P2.54mm_Vertical, F.Cu at (191.3, 105.3)
- added J3: Conn_01x08, Connector_PinSocket_2.54mm:PinSocket_1x08_P2.54mm_Vertical, F.Cu at (209.1, 132.3)
- added J4: Conn_02x08_Counter_Clockwise, Connector_PinHeader_2.54mm:PinHeader_2x08_P2.54mm_Vertical, F.Cu at (158.5, 114.0)
- added R1: R1K, Resistor_SMD:R_0603_1608Metric_Pad1.05x0.95mm_HandSolder, F.Cu at (170.4, 113.5)
- added U1: LM1117-3.3, Package_TO_SOT_SMD:SOT-223, F.Cu at (168.5, 107.8)
- R4, R6: footprint Resistor_SMD:R_0603_1608Metric -> Resistor_SMD:R_0603_1608Metric_Pad1.05x0.95mm_HandSolder
- moved R6 14.6 mm to (182.3, 118.0), turned to 270 degrees
- moved R4 9.89 mm to (182.3, 121.8), turned to 90 degrees
- moved Boot1 2.15 mm to (178.3, 122.0)
- moved Reset1 1.77 mm to (178.3, 118.0)
- moved U4 0.50 mm to (199.1, 118.8)
Connections:
- net Net-(J4-Pad14) renamed /di
- net Net-(R1-Pad2) renamed /cs
- net Net-(U4-Pad12) renamed /miso
- net Net-(U4-Pad13) renamed /sck
- net Net-(U4-Pad14) renamed /ci
- net Net-(U4-Pad16) renamed /mosi
- U4 pad 29: Net-(J5-Pad8) -> /io5_cs
- U4 pad 30: Net-(J5-Pad7) -> /io18_sck
- U4 pad 31: Net-(J5-Pad6) -> /io19_miso
- U4 pad 33: Net-(J5-Pad5) -> /qhd
- U4 pad 36: Net-(J5-Pad2) -> /qwp
- U4 pad 37: Net-(J5-Pad1) -> /io23_mosi
Other:
- board size 50 x 31 mm -> 56.2 x 31 mm
